File: Test Harness board - kicad 5.99/Left.kicad_sch (KiCad schematic)
At the start: 126 parts

Commit message: oops, had the connector on the wrong side !
Parts:
- D_A0, D_A1, D_A10, D_A11, D_A12, D_A13, D_A14, D_A15, D_A16, D_A17, D_A18, D_A19, D_A2, D_A20, D_A21, D_A3, D_A4, D_A5, D_A6, D_A7, D_A8, D_A9, D_D0, D_D1, D_D2, D_D3, D_D4, D_D5, D_D6, D_D7, D_IR2, D_IR3, D_L0, D_L1, D_L10, D_L11, D_L12, D_L13, D_L14, D_L15, D_L2, D_L3, D_L4, D_L5, D_L6, D_L7, D_L8, D_L9, D_MAR0, D_MAR1, D_MAR10, D_MAR11, D_MAR12, D_MAR13, D_MAR14, D_MAR15, D_MAR2, D_MAR3, D_MAR4, D_MAR5, D_MAR6, D_MAR7, D_MAR8, D_MAR9, D_MEMORY1, D_MEMREF1, D_XL_MDR_HI1, D_XL_MDR_LO1, D__IR1, D__IRQ4, D__PSEL1, D__RD1, D__RESET1, D__STOP_CLK1, D__WR1: footprint LED_SMD:LED_1206_3216Metric_Castellated -> LED_SMD:LED_0805_2012Metric
- UL1, UL3, UL4, UL5: footprint Package_SO:SOIC-28W_7.5x17.9mm_P1.27mm -> Package_SO:TSSOP-28_4.4x9.7mm_P0.65mm
- UL1_1, UL1_2, UL2_1, UL2_2, UL3_1, UL3_2, UL4_1, UL4_2, UL5_1, UL5_2: footprint Package_SO:SOIC-20W_7.5x12.8mm_P1.27mm -> Package_SO:TSSOP-20_4.4x6.5mm_P0.65mm
