File: Test_harness/Test Harness board.kicad_sch (KiCad schematic)
At the start: 5 parts, among them U1 TCA9548APWR

Commit message: added a bunch of things, including board under test power control
Parts:
- added CBP1: 1µF, Capacitor_SMD:C_0805_2012Metric, symbol Device:C_Small
- added CBP2: 0.1µF, Capacitor_SMD:C_0805_2012Metric, symbol Device:C_Small
- added CBP3: 120µF, Capacitor_SMD:CP_Elec_6.3x9.9, symbol Device:CP1_Small
- added DBP1: LED_Small, LED_SMD:LED_0805_2012Metric, symbol Device:LED_Small
- added RBP1: 10kΩ, Resistor_SMD:R_0805_2012Metric, symbol Device:R
- added RBP2, RBP3: 1kΩ, Resistor_SMD:R_0805_2012Metric, symbol Device:R
- added UBP1: AP22814AW5, Package_TO_SOT_SMD:SOT-23-5, symbol Power_Management:AP22814AW5
Connections:
- net +5V: now also CBP1.1, RBP1.1, UBP1.5 (IN)
- net GND: now also CBP1.2, CBP2.2, CBP3.2, DBP1.1 (K), RBP3.2, UBP1.2 (GND)
- net PWR_BOARD_ON: now reaches A1.5 (D2)
- net PWR_BOARD_ON: now also RBP3.1, UBP1.4 (EN)
- new net: DBP1.2 (A), RBP2.1
- new net: RBP1.2, UBP1.3 (~FLG)
- new net BRD_POWER: CBP2.1, CBP3.1, RBP2.2, UBP1.1 (OUT)

Commit message: more fixes
Connections:
- net SCL_1 renamed SDA_0
Other:
- sheet Left connector ports: added SCL, SDA; removed none
Changed lines of the file:
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@@
     (effects (font (size 1.27 1.27)) (justify left bottom))
   )
-  (label "SCL_1" (at 49.53 118.11 0)
+  (label "SDA_0" (at 49.53 118.11 0)
     (effects (font (size 1.27 1.27)) (justify left bottom))
   )
@@
   )
   (label "PWR_BOARD_ON" (at 97.79 67.31 180)
+    (effects (font (size 1.27 1.27)) (justify right bottom))
+  )
+  (label "SDA_0" (at 176.53 24.13 180)
+    (effects (font (size 1.27 1.27)) (justify right bottom))
+  )
+  (label "SCL_0" (at 176.53 26.67 180)
     (effects (font (size 1.27 1.27)) (justify right bottom))
   )
@@
       (effects (font (size 1.27 1.27)) (justify left top))
     )
+    (pin "SDA" input (at 176.53 24.13 180)
+      (effects (font (size 1.27 1.27)) (justify left))
+    )
+    (pin "SCL" input (at 176.53 26.67 180)
+      (effects (font (size 1.27 1.27)) (justify left))
+    )
   )
   (symbol_instances
@@
     )
     (path "/0bb7ffcb-56f8-4343-bb38-9a762c1c79b6/d347ac01-2758-4fd6-be7e-17ff760dc997"
-      (reference "RNL2_2_1") (unit 1) (value "R_Pack04") (footprint "Resistor_SMD:R_Array_Convex_4x1206")
+      (reference "RNL2_2_1") (unit 1) (value "1kΩ") (footprint "Resistor_SMD:R_Array_Convex_4x1206")
     )
     (path "/0bb7ffcb-56f8-4343-bb38-9a762c1c79b6/f54264b3-e6e5-44ec-8677-1ead6d88cfe1"
