File: ALU/ALU-v2.0/ALU.kicad_sch (KiCad schematic)
At the start: 50 parts, among them U1 74F381, U10 74ACT244, U11 74ACT244, U12 74ACT04, U13 74ACT00, U14 74ACT32, U15 74ACT02, U16 74ACT157, U17 74ACT153, U18 74ACT153, U19 74ACT08, U2 74F381, U20 74ACT20, U21 74ACT02, U22 74ACT02, U3 74F381, U4 74F382, U5 74F382, U6 74F182, U7 74ACT244, U8 74ACT244, U9 74ACT244

Commit message: change all caps to 0805
Parts:
- C1, C10, C11, C12, C13, C14, C15, C16, C17, C18, C19, C2, C20, C21, C22, C23, C24, C25, C26, C27, C28, C3, C4, C5, C6, C7, C8, C9: footprint Capacitor_SMD:C_1206_3216Metric -> Capacitor_SMD:C_0805_2012Metric
Changed lines of the file:
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@@
   (junction (at 367.03 233.68) (diameter 1.016) (color 0 0 0 0))
   (no_connect (at 224.79 49.53))
+  (no_connect (at 130.81 119.38))
+  (no_connect (at 69.85 111.76))
+  (no_connect (at 224.79 52.07))
   (no_connect (at 224.79 46.99))
-  (no_connect (at 130.81 119.38))
   (no_connect (at 130.81 121.92))
-  (no_connect (at 224.79 52.07))
-  (no_connect (at 69.85 111.76))
   (wire (pts (xy 21.59 269.24) (xy 30.48 269.24))
     (stroke (width 0) (type solid) (color 0 0 0 0))
@@
       (effects (font (size 1.27 1.27)) (justify left))
     )
-    (property "Footprint" "Capacitor_SMD:C_1206_3216Metric" (id 2) (at 22.5552 276.86 0)
+    (property "Footprint" "Capacitor_SMD:C_0805_2012Metric" (id 2) (at 22.5552 276.86 0)
       (effects (font (size 1.27 1.27)) hide)
     )
@@
       (effects (font (size 1.27 1.27)) (justify left))
     )
-    (property "Footprint" "Capacitor_SMD:C_1206_3216Metric" (id 2) (at 31.4452 276.86 0)
+    (property "Footprint" "Capacitor_SMD:C_0805_2012Metric" (id 2) (at 31.4452 276.86 0)
       (effects (font (size 1.27 1.27)) hide)
     )
@@
       (effects (font (size 1.27 1.27)) (justify left))
     )
-    (property "Footprint" "Capacitor_SMD:C_1206_3216Metric" (id 2) (at 40.3352 276.86 0)
+    (property "Footprint" "Capacitor_SMD:C_0805_2012Metric" (id 2) (at 40.3352 276.86 0)
       (effects (font (size 1.27 1.27)) hide)
     )
@@
       (effects (font (size 1.27 1.27)) (justify left))
     )
-    (property "Footprint" "Capacitor_SMD:C_1206_3216Metric" (id 2) (at 49.2252 276.86 0)
+    (property "Footprint" "Capacitor_SMD:C_0805_2012Metric" (id 2) (at 49.2252 276.86 0)
       (effects (font (size 1.27 1.27)) hide)
     )
@@
       (effects (font (size 1.27 1.27)) (justify left))
     )
-    (property "Footprint" "Capacitor_SMD:C_1206_3216Metric" (id 2) (at 58.1152 276.86 0)
+    (property "Footprint" "Capacitor_SMD:C_0805_2012Metric" (id 2) (at 58.1152 276.86 0)
       (effects (font (size 1.27 1.27)) hide)
     )
@@
       (effects (font (size 1.27 1.27)) (justify left))
     )
-    (property "Footprint" "Capacitor_SMD:C_1206_3216Metric" (id 2) (at 67.0052 276.86 0)
+    (property "Footprint" "Capacitor_SMD:C_0805_2012Metric" (id 2) (at 67.0052 276.86 0)
       (effects (font (size 1.27 1.27)) hide)
     )
@@
       (effects (font (size 1.27 1.27)) (justify left))
     )
-    (property "Footprint" "Capacitor_SMD:C_1206_3216Metric" (id 2) (at 75.8952 276.86 0)
+    (property "Footprint" "Capacitor_SMD:C_0805_2012Metric" (id 2) (at 75.8952 276.86 0)
       (effects (font (size 1.27 1.27)) hide)
     )
@@
       (effects (font (size 1.27 1.27)) (justify left))
     )
-    (property "Footprint" "Capacitor_SMD:C_1206_3216Metric" (id 2) (at 84.7852 276.86 0)
+    (property "Footprint" "Capacitor_SMD:C_0805_2012Metric" (id 2) (at 84.7852 276.86 0)
       (effects (font (size 1.27 1.27)) hide)
     )
@@
       (effects (font (size 1.27 1.27)) (justify left))
     )
-    (property "Footprint" "Capacitor_SMD:C_1206_3216Metric" (id 2) (at 93.6752 276.86 0)
+    (property "Footprint" "Capacitor_SMD:C_0805_2012Metric" (id 2) (at 93.6752 276.86 0)
       (effects (font (size 1.27 1.27)) hide)
     )
@@
       (effects (font (size 1.27 1.27)) (justify left))
     )
-    (property "Footprint" "Capacitor_SMD:C_1206_3216Metric" (id 2) (at 102.5652 276.86 0)
+    (property "Footprint" "Capacitor_SMD:C_0805_2012Metric" (id 2) (at 102.5652 276.86 0)
       (effects (font (size 1.27 1.27)) hide)
     )
@@
       (effects (font (size 1.27 1.27)) (justify left))
     )
-    (property "Footprint" "Capacitor_SMD:C_1206_3216Metric" (id 2) (at 111.4552 276.86 0)
+    (property "Footprint" "Capacitor_SMD:C_0805_2012Metric" (id 2) (at 111.4552 276.86 0)
       (effects (font (size 1.27 1.27)) hide)
     )
@@
       (effects (font (size 1.27 1.27)) (justify left))
     )
-    (property "Footprint" "Capacitor_SMD:C_1206_3216Metric" (id 2) (at 120.3452 276.86 0)
+    (property "Footprint" "Capacitor_SMD:C_0805_2012Metric" (id 2) (at 120.3452 276.86 0)
       (effects (font (size 1.27 1.27)) hide)
     )
@@
       (effects (font (size 1.27 1.27)) (justify left))
     )
-    (property "Footprint" "Capacitor_SMD:C_1206_3216Metric" (id 2) (at 129.2352 276.86 0)
+    (property "Footprint" "Capacitor_SMD:C_0805_2012Metric" (id 2) (at 129.2352 276.86 0)
       (effects (font (size 1.27 1.27)) hide)
     )
@@
       (effects (font (size 1.27 1.27)) (justify left))
     )
-    (property "Footprint" "Capacitor_SMD:C_1206_3216Metric" (id 2) (at 138.1252 276.86 0)
+    (property "Footprint" "Capacitor_SMD:C_0805_2012Metric" (id 2) (at 138.1252 276.86 0)
       (effects (font (size 1.27 1.27)) hide)
     )
@@
       (effects (font (size 1.27 1.27)) (justify left))
     )
-    (property "Footprint" "Capacitor_SMD:C_1206_3216Metric" (id 2) (at 147.0152 276.86 0)
+    (property "Footprint" "Capacitor_SMD:C_0805_2012Metric" (id 2) (at 147.0152 276.86 0)
       (effects (font (size 1.27 1.27)) hide)
     )
@@
       (effects (font (size 1.27 1.27)) (justify left))
     )
-    (property "Footprint" "Capacitor_SMD:C_1206_3216Metric" (id 2) (at 155.9052 276.86 0)
+    (property "Footprint" "Capacitor_SMD:C_0805_2012Metric" (id 2) (at 155.9052 276.86 0)
       (effects (font (size 1.27 1.27)) hide)
     )
@@
       (effects (font (size 1.27 1.27)) (justify left))
     )
-    (property "Footprint" "Capacitor_SMD:C_1206_3216Metric" (id 2) (at 164.7952 276.86 0)
+    (property "Footprint" "Capacitor_SMD:C_0805_2012Metric" (id 2) (at 164.7952 276.86 0)
       (effects (font (size 1.27 1.27)) hide)
     )
@@
       (effects (font (size 1.27 1.27)) (justify left))
     )
-    (property "Footprint" "Capacitor_SMD:C_1206_3216Metric" (id 2) (at 173.6852 276.86 0)
+    (property "Footprint" "Capacitor_SMD:C_0805_2012Metric" (id 2) (at 173.6852 276.86 0)
       (effects (font (size 1.27 1.27)) hide)
     )
@@
       (effects (font (size 1.27 1.27)) (justify left))
     )
-    (property "Footprint" "Capacitor_SMD:C_1206_3216Metric" (id 2) (at 182.5752 276.86 0)
+    (property "Footprint" "Capacitor_SMD:C_0805_2012Metric" (id 2) (at 182.5752 276.86 0)
       (effects (font (size 1.27 1.27)) hide)
     )
@@
       (effects (font (size 1.27 1.27)) (justify left))
     )
-    (property "Footprint" "Capacitor_SMD:C_1206_3216Metric" (id 2) (at 191.4652 276.86 0)
+    (property "Footprint" "Capacitor_SMD:C_0805_2012Metric" (id 2) (at 191.4652 276.86 0)
       (effects (font (size 1.27 1.27)) hide)
     )
@@
       (effects (font (size 1.27 1.27)) (justify left))
     )
-    (property "Footprint" "Capacitor_SMD:C_1206_3216Metric" (id 2) (at 200.3552 276.86 0)
+    (property "Footprint" "Capacitor_SMD:C_0805_2012Metric" (id 2) (at 200.3552 276.86 0)
       (effects (font (size 1.27 1.27)) hide)
     )
@@
       (effects (font (size 1.27 1.27)) (justify left))
     )
-    (property "Footprint" "Capacitor_SMD:C_1206_3216Metric" (id 2) (at 209.2452 276.86 0)
+    (property "Footprint" "Capacitor_SMD:C_0805_2012Metric" (id 2) (at 209.2452 276.86 0)
       (effects (font (size 1.27 1.27)) hide)
     )
@@
       (effects (font (size 1.27 1.27)) (justify left))
     )
-    (property "Footprint" "Capacitor_SMD:C_1206_3216Metric" (id 2) (at 218.1352 276.86 0)
+    (property "Footprint" "Capacitor_SMD:C_0805_2012Metric" (id 2) (at 218.1352 276.86 0)
       (effects (font (size 1.27 1.27)) hide)
     )
@@
       (effects (font (size 1.27 1.27)) (justify left))
     )
-    (property "Footprint" "Capacitor_SMD:C_1206_3216Metric" (id 2) (at 227.0252 276.86 0)
+    (property "Footprint" "Capacitor_SMD:C_0805_2012Metric" (id 2) (at 227.0252 276.86 0)
       (effects (font (size 1.27 1.27)) hide)
     )
@@
       (effects (font (size 1.27 1.27)) (justify left))
     )
-    (property "Footprint" "Capacitor_SMD:C_1206_3216Metric" (id 2) (at 235.9152 276.86 0)
+    (property "Footprint" "Capacitor_SMD:C_0805_2012Metric" (id 2) (at 235.9152 276.86 0)
       (effects (font (size 1.27 1.27)) hide)
     )
@@
       (effects (font (size 1.27 1.27)) (justify left))
     )
-    (property "Footprint" "Capacitor_SMD:C_1206_3216Metric" (id 2) (at 244.8052 276.86 0)
+    (property "Footprint" "Capacitor_SMD:C_0805_2012Metric" (id 2) (at 244.8052 276.86 0)
       (effects (font (size 1.27 1.27)) hide)
     )
@@
       (effects (font (size 1.27 1.27)) (justify left))
     )
-    (property "Footprint" "Capacitor_SMD:C_1206_3216Metric" (id 2) (at 253.6952 276.86 0)
+    (property "Footprint" "Capacitor_SMD:C_0805_2012Metric" (id 2) (at 253.6952 276.86 0)
       (effects (font (size 1.27 1.27)) hide)
     )
@@
       (effects (font (size 1.27 1.27)) (justify left))
     )
-    (property "Footprint" "Capacitor_SMD:C_1206_3216Metric" (id 2) (at 262.5852 276.86 0)
-      (effects (font (size 1.27 1.27)) hide)
-    )
+    (property "Footprint" "Capacitor_SMD:C_0805_2012Metric" (id 2) (at 262.5852 276.86 0)
+      (effects (font (size 1.27 1.27)) hide)
+    )
