File: ALU/ALU-v2.0/Genreral registers.kicad_sch (KiCad schematic)
At the start: 32 parts, among them U29 74ACT374, U30 74ACT374, U31 74ACT374, U32 74ACT374, U33 74ACT374, U34 74ACT374, U35 74ACT374, U36 74ACT374, U37 74ACT374, U38 74ACT374, U39 74ACT374, U40 74ACT374, U41 74ACT374, U42 74ACT374, U43 74ACT374, U44 74ACT374

Commit message: change all caps to 0805
Parts:
- C29, C30, C31, C32, C33, C34, C35, C36, C37, C38, C39, C40, C41, C42, C43, C44: footprint Capacitor_SMD:C_1206_3216Metric -> Capacitor_SMD:C_0805_2012Metric
Changed lines of the file:
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@@
       (effects (font (size 1.27 1.27)) (justify left))
     )
-    (property "Footprint" "Capacitor_SMD:C_1206_3216Metric" (id 2) (at 100.0252 171.45 0)
+    (property "Footprint" "Capacitor_SMD:C_0805_2012Metric" (id 2) (at 100.0252 171.45 0)
       (effects (font (size 1.27 1.27)) hide)
     )
@@
       (effects (font (size 1.27 1.27)) (justify left))
     )
-    (property "Footprint" "Capacitor_SMD:C_1206_3216Metric" (id 2) (at 110.1852 171.45 0)
+    (property "Footprint" "Capacitor_SMD:C_0805_2012Metric" (id 2) (at 110.1852 171.45 0)
       (effects (font (size 1.27 1.27)) hide)
     )
@@
       (effects (font (size 1.27 1.27)) (justify left))
     )
-    (property "Footprint" "Capacitor_SMD:C_1206_3216Metric" (id 2) (at 120.3452 171.45 0)
+    (property "Footprint" "Capacitor_SMD:C_0805_2012Metric" (id 2) (at 120.3452 171.45 0)
       (effects (font (size 1.27 1.27)) hide)
     )
@@
       (effects (font (size 1.27 1.27)) (justify left))
     )
-    (property "Footprint" "Capacitor_SMD:C_1206_3216Metric" (id 2) (at 130.5052 171.45 0)
+    (property "Footprint" "Capacitor_SMD:C_0805_2012Metric" (id 2) (at 130.5052 171.45 0)
       (effects (font (size 1.27 1.27)) hide)
     )
@@
       (effects (font (size 1.27 1.27)) (justify left))
     )
-    (property "Footprint" "Capacitor_SMD:C_1206_3216Metric" (id 2) (at 140.6652 171.45 0)
+    (property "Footprint" "Capacitor_SMD:C_0805_2012Metric" (id 2) (at 140.6652 171.45 0)
       (effects (font (size 1.27 1.27)) hide)
     )
@@
       (effects (font (size 1.27 1.27)) (justify left))
     )
-    (property "Footprint" "Capacitor_SMD:C_1206_3216Metric" (id 2) (at 150.8252 171.45 0)
+    (property "Footprint" "Capacitor_SMD:C_0805_2012Metric" (id 2) (at 150.8252 171.45 0)
       (effects (font (size 1.27 1.27)) hide)
     )
@@
       (effects (font (size 1.27 1.27)) (justify left))
     )
-    (property "Footprint" "Capacitor_SMD:C_1206_3216Metric" (id 2) (at 160.9852 171.45 0)
+    (property "Footprint" "Capacitor_SMD:C_0805_2012Metric" (id 2) (at 160.9852 171.45 0)
       (effects (font (size 1.27 1.27)) hide)
     )
@@
       (effects (font (size 1.27 1.27)) (justify left))
     )
-    (property "Footprint" "Capacitor_SMD:C_1206_3216Metric" (id 2) (at 171.1452 171.45 0)
+    (property "Footprint" "Capacitor_SMD:C_0805_2012Metric" (id 2) (at 171.1452 171.45 0)
       (effects (font (size 1.27 1.27)) hide)
     )
@@
       (effects (font (size 1.27 1.27)) (justify left))
     )
-    (property "Footprint" "Capacitor_SMD:C_1206_3216Metric" (id 2) (at 181.3052 171.45 0)
+    (property "Footprint" "Capacitor_SMD:C_0805_2012Metric" (id 2) (at 181.3052 171.45 0)
       (effects (font (size 1.27 1.27)) hide)
     )
@@
       (effects (font (size 1.27 1.27)) (justify left))
     )
-    (property "Footprint" "Capacitor_SMD:C_1206_3216Metric" (id 2) (at 191.4652 171.45 0)
+    (property "Footprint" "Capacitor_SMD:C_0805_2012Metric" (id 2) (at 191.4652 171.45 0)
       (effects (font (size 1.27 1.27)) hide)
     )
@@
       (effects (font (size 1.27 1.27)) (justify left))
     )
-    (property "Footprint" "Capacitor_SMD:C_1206_3216Metric" (id 2) (at 201.6252 171.45 0)
+    (property "Footprint" "Capacitor_SMD:C_0805_2012Metric" (id 2) (at 201.6252 171.45 0)
       (effects (font (size 1.27 1.27)) hide)
     )
@@
       (effects (font (size 1.27 1.27)) (justify left))
     )
-    (property "Footprint" "Capacitor_SMD:C_1206_3216Metric" (id 2) (at 211.7852 171.45 0)
+    (property "Footprint" "Capacitor_SMD:C_0805_2012Metric" (id 2) (at 211.7852 171.45 0)
       (effects (font (size 1.27 1.27)) hide)
     )
@@
       (effects (font (size 1.27 1.27)) (justify left))
     )
-    (property "Footprint" "Capacitor_SMD:C_1206_3216Metric" (id 2) (at 221.9452 171.45 0)
+    (property "Footprint" "Capacitor_SMD:C_0805_2012Metric" (id 2) (at 221.9452 171.45 0)
       (effects (font (size 1.27 1.27)) hide)
     )
@@
       (effects (font (size 1.27 1.27)) (justify left))
     )
-    (property "Footprint" "Capacitor_SMD:C_1206_3216Metric" (id 2) (at 232.1052 171.45 0)
+    (property "Footprint" "Capacitor_SMD:C_0805_2012Metric" (id 2) (at 232.1052 171.45 0)
       (effects (font (size 1.27 1.27)) hide)
     )
@@
       (effects (font (size 1.27 1.27)) (justify left))
     )
-    (property "Footprint" "Capacitor_SMD:C_1206_3216Metric" (id 2) (at 242.2652 171.45 0)
+    (property "Footprint" "Capacitor_SMD:C_0805_2012Metric" (id 2) (at 242.2652 171.45 0)
       (effects (font (size 1.27 1.27)) hide)
     )
@@
       (effects (font (size 1.27 1.27)) (justify left))
     )
-    (property "Footprint" "Capacitor_SMD:C_1206_3216Metric" (id 2) (at 252.4252 171.45 0)
-      (effects (font (size 1.27 1.27)) hide)
-    )
+    (property "Footprint" "Capacitor_SMD:C_0805_2012Metric" (id 2) (at 252.4252 171.45 0)
+      (effects (font (size 1.27 1.27)) hide)
+    )
