File: ALU/ALU-v2.0/Immediate Register.kicad_sch (KiCad schematic)
At the start: 4 parts, among them U45 74ACT244, U46 74ACT244

Commit message: change all caps to 0805
Parts:
- C45, C46: footprint Capacitor_SMD:C_1206_3216Metric -> Capacitor_SMD:C_0805_2012Metric
Changed lines of the file:
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@@
       (effects (font (size 1.27 1.27)) (justify left))
     )
-    (property "Footprint" "Capacitor_SMD:C_1206_3216Metric" (id 2) (at 27.6352 153.67 0)
+    (property "Footprint" "Capacitor_SMD:C_0805_2012Metric" (id 2) (at 27.6352 153.67 0)
       (effects (font (size 1.27 1.27)) hide)
     )
@@
       (effects (font (size 1.27 1.27)) (justify left))
     )
-    (property "Footprint" "Capacitor_SMD:C_1206_3216Metric" (id 2) (at 36.5252 153.67 0)
+    (property "Footprint" "Capacitor_SMD:C_0805_2012Metric" (id 2) (at 36.5252 153.67 0)
       (effects (font (size 1.27 1.27)) hide)
     )
