File: ALU/ALU-v2.0/MAR.kicad_sch (KiCad schematic)
At the start: 8 parts, among them U47 74ACT273, U48 74ACT273, U49 74ACT244, U50 74ACT244

Commit message: change all caps to 0805
Parts:
- C62, C63, C64, C65: footprint Capacitor_SMD:C_1206_3216Metric -> Capacitor_SMD:C_0805_2012Metric
Changed lines of the file:
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@@
       (effects (font (size 1.27 1.27)) (justify left))
     )
-    (property "Footprint" "Capacitor_SMD:C_1206_3216Metric" (id 2) (at 44.1452 170.18 0)
+    (property "Footprint" "Capacitor_SMD:C_0805_2012Metric" (id 2) (at 44.1452 170.18 0)
       (effects (font (size 1.27 1.27)) hide)
     )
@@
       (effects (font (size 1.27 1.27)) (justify left))
     )
-    (property "Footprint" "Capacitor_SMD:C_1206_3216Metric" (id 2) (at 54.3052 170.18 0)
+    (property "Footprint" "Capacitor_SMD:C_0805_2012Metric" (id 2) (at 54.3052 170.18 0)
       (effects (font (size 1.27 1.27)) hide)
     )
@@
       (effects (font (size 1.27 1.27)) (justify left))
     )
-    (property "Footprint" "Capacitor_SMD:C_1206_3216Metric" (id 2) (at 64.4652 170.18 0)
+    (property "Footprint" "Capacitor_SMD:C_0805_2012Metric" (id 2) (at 64.4652 170.18 0)
       (effects (font (size 1.27 1.27)) hide)
     )
@@
       (effects (font (size 1.27 1.27)) (justify left))
     )
-    (property "Footprint" "Capacitor_SMD:C_1206_3216Metric" (id 2) (at 74.6252 170.18 0)
+    (property "Footprint" "Capacitor_SMD:C_0805_2012Metric" (id 2) (at 74.6252 170.18 0)
       (effects (font (size 1.27 1.27)) hide)
     )
