File: ALU/ALU-v2.0/MDR.kicad_sch (KiCad schematic)
At the start: 31 parts, among them U12 74ACT04, U51 74ACT157, U52 74ACT157, U53 74ACT273, U54 74ACT273, U55 74ACT244, U56 74ACT244, U57 74ACT244, U58 74ACT244, U59 74ACT244, U60 74ACT244, U61 74ACT245, U62 74ACT153, U63 74ACT153, U64 74ACT153, U65 74ACT153

Commit message: change all caps to 0805
Parts:
- C47, C48, C49, C50, C51, C52, C53, C54, C55, C56, C57, C58, C59, C60, C61: footprint Capacitor_SMD:C_1206_3216Metric -> Capacitor_SMD:C_0805_2012Metric
Changed lines of the file:
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@@
       (effects (font (size 1.27 1.27)) (justify left))
     )
-    (property "Footprint" "Capacitor_SMD:C_1206_3216Metric" (id 2) (at 206.7052 240.03 0)
+    (property "Footprint" "Capacitor_SMD:C_0805_2012Metric" (id 2) (at 206.7052 240.03 0)
       (effects (font (size 1.27 1.27)) hide)
     )
@@
       (effects (font (size 1.27 1.27)) (justify left))
     )
-    (property "Footprint" "Capacitor_SMD:C_1206_3216Metric" (id 2) (at 215.5952 240.03 0)
+    (property "Footprint" "Capacitor_SMD:C_0805_2012Metric" (id 2) (at 215.5952 240.03 0)
       (effects (font (size 1.27 1.27)) hide)
     )
@@
       (effects (font (size 1.27 1.27)) (justify left))
     )
-    (property "Footprint" "Capacitor_SMD:C_1206_3216Metric" (id 2) (at 224.4852 240.03 0)
+    (property "Footprint" "Capacitor_SMD:C_0805_2012Metric" (id 2) (at 224.4852 240.03 0)
       (effects (font (size 1.27 1.27)) hide)
     )
@@
       (effects (font (size 1.27 1.27)) (justify left))
     )
-    (property "Footprint" "Capacitor_SMD:C_1206_3216Metric" (id 2) (at 233.3752 240.03 0)
+    (property "Footprint" "Capacitor_SMD:C_0805_2012Metric" (id 2) (at 233.3752 240.03 0)
       (effects (font (size 1.27 1.27)) hide)
     )
@@
       (effects (font (size 1.27 1.27)) (justify left))
     )
-    (property "Footprint" "Capacitor_SMD:C_1206_3216Metric" (id 2) (at 242.2652 240.03 0)
+    (property "Footprint" "Capacitor_SMD:C_0805_2012Metric" (id 2) (at 242.2652 240.03 0)
       (effects (font (size 1.27 1.27)) hide)
     )
@@
       (effects (font (size 1.27 1.27)) (justify left))
     )
-    (property "Footprint" "Capacitor_SMD:C_1206_3216Metric" (id 2) (at 251.1552 240.03 0)
+    (property "Footprint" "Capacitor_SMD:C_0805_2012Metric" (id 2) (at 251.1552 240.03 0)
       (effects (font (size 1.27 1.27)) hide)
     )
@@
       (effects (font (size 1.27 1.27)) (justify left))
     )
-    (property "Footprint" "Capacitor_SMD:C_1206_3216Metric" (id 2) (at 260.0452 240.03 0)
+    (property "Footprint" "Capacitor_SMD:C_0805_2012Metric" (id 2) (at 260.0452 240.03 0)
       (effects (font (size 1.27 1.27)) hide)
     )
@@
       (effects (font (size 1.27 1.27)) (justify left))
     )
-    (property "Footprint" "Capacitor_SMD:C_1206_3216Metric" (id 2) (at 268.9352 240.03 0)
+    (property "Footprint" "Capacitor_SMD:C_0805_2012Metric" (id 2) (at 268.9352 240.03 0)
       (effects (font (size 1.27 1.27)) hide)
     )
@@
       (effects (font (size 1.27 1.27)) (justify left))
     )
-    (property "Footprint" "Capacitor_SMD:C_1206_3216Metric" (id 2) (at 277.8252 240.03 0)
+    (property "Footprint" "Capacitor_SMD:C_0805_2012Metric" (id 2) (at 277.8252 240.03 0)
       (effects (font (size 1.27 1.27)) hide)
     )
@@
       (effects (font (size 1.27 1.27)) (justify left))
     )
-    (property "Footprint" "Capacitor_SMD:C_1206_3216Metric" (id 2) (at 286.7152 240.03 0)
+    (property "Footprint" "Capacitor_SMD:C_0805_2012Metric" (id 2) (at 286.7152 240.03 0)
       (effects (font (size 1.27 1.27)) hide)
     )
@@
       (effects (font (size 1.27 1.27)) (justify left))
     )
-    (property "Footprint" "Capacitor_SMD:C_1206_3216Metric" (id 2) (at 295.6052 240.03 0)
+    (property "Footprint" "Capacitor_SMD:C_0805_2012Metric" (id 2) (at 295.6052 240.03 0)
       (effects (font (size 1.27 1.27)) hide)
     )
@@
       (effects (font (size 1.27 1.27)) (justify left))
     )
-    (property "Footprint" "Capacitor_SMD:C_1206_3216Metric" (id 2) (at 304.4952 240.03 0)
+    (property "Footprint" "Capacitor_SMD:C_0805_2012Metric" (id 2) (at 304.4952 240.03 0)
       (effects (font (size 1.27 1.27)) hide)
     )
@@
       (effects (font (size 1.27 1.27)) (justify left))
     )
-    (property "Footprint" "Capacitor_SMD:C_1206_3216Metric" (id 2) (at 313.3852 240.03 0)
+    (property "Footprint" "Capacitor_SMD:C_0805_2012Metric" (id 2) (at 313.3852 240.03 0)
       (effects (font (size 1.27 1.27)) hide)
     )
@@
       (effects (font (size 1.27 1.27)) (justify left))
     )
-    (property "Footprint" "Capacitor_SMD:C_1206_3216Metric" (id 2) (at 322.2752 240.03 0)
+    (property "Footprint" "Capacitor_SMD:C_0805_2012Metric" (id 2) (at 322.2752 240.03 0)
       (effects (font (size 1.27 1.27)) hide)
     )
@@
       (effects (font (size 1.27 1.27)) (justify left))
     )
-    (property "Footprint" "Capacitor_SMD:C_1206_3216Metric" (id 2) (at 331.1652 240.03 0)
-      (effects (font (size 1.27 1.27)) hide)
-    )
+    (property "Footprint" "Capacitor_SMD:C_0805_2012Metric" (id 2) (at 331.1652 240.03 0)
+      (effects (font (size 1.27 1.27)) hide)
+    )
