File: Control Card/microcode.kicad_sch (KiCad schematic)
At the start: 36 parts, among them U1 CY7C1021D, U10 74ACT273, U100 74LVC1G08, U101 74LVC1G32, U102 74LVC2G157, U11 74ACT151, U110 74ACT244, U111 74ACT374, U112 74ACT374, U113 74ACT374, U114 74ACT374, U115 74ACT374, U116 74ACT374, U117 74ACT374, U118 74ACT374, U119 74ACT374, U12 74ACT86, U13 74ACT32, U14 74ACT04, U15 74ACT153, U16 74ACT153, U17 74ACT153, U18 74ACT153, U2 CY7C1021D, U20 74ACT02, U21 74ACT20, U24 74ACT30, U3 CY7C1021D, U44 74ACT11, U5 74ACT273, U53 74ACT04, U6 74ACT273, U61 74ACT32, U7 74ACT273, U8 74ACT273, U9 74ACT273

Commit message: add lots of nets to the Din connectors
Parts:
- added U19: 74ACT273, Package_SO:SOIC-20W_7.5x12.8mm_P1.27mm, symbol 74xx:74LS273
Connections:
- net +5V: now also U19.20 (VCC)
- net GND: now also U19.1 (~Mr), U19.10 (GND), U19.11 (Cp)
- net IR0: now also U19.19 (Q7)
- net IR1: now also U19.16 (Q6)
- net IR2: now also U19.15 (Q5)
- net IR3: now also U19.12 (Q4)
- net IR4: now also U19.9 (Q3)
- net IR5: now also U19.6 (Q2)
- net IR6: now also U19.5 (Q1)
- net IR7: now also U19.2 (Q0)
- net i_DBUS0: now also U19.18 (D7)
- net i_DBUS1: now also U19.17 (D6)
- net i_DBUS2: now also U19.14 (D5)
- net i_DBUS3: now also U19.13 (D4)
- net i_DBUS4: now also U19.8 (D3)
- net i_DBUS5: now also U19.7 (D2)
- net i_DBUS6: now also U19.4 (D1)
- net i_DBUS7: now also U19.3 (D0)
Other:
- note added: "Instruction Register"
- note added: "Stores the micro-instruction that is to be written to the µcode store"
- note added: "Stores the µcode write access bits"
- note added: "µcode address to be written"
- note added: "µcode current execution page register"
